File: Eagle/ENC_BOARD_V01/ENC_BOARD_V01.brd (EAGLE design)
At the start: 79 x 56 mm, 13 parts, among them X1 057-026-1

Commit message: Updated Encoder Board
Parts:
- moved EN1 20.0 mm to (69.5, 40.0)
- moved EN2 20.0 mm to (69.5, 20.0)
Routing:
- net N$3: track 26.9 -> 49.7 mm
- net N$1: track 13.4 -> 32.2 mm
- net N$6: track 50.6 -> 33.4 mm
- net N$2: track 19.5 -> 36.4 mm
- net N$4: track 34.9 -> 18.8 mm
- net N$5: track 37.3 -> 23.6 mm
- net N$13: track 32.9 -> 40.6 mm, vias 0 -> 1
- net N$7: track 27.8 -> 28.8 mm
- net N$17: track 8.71 -> 9.61 mm
- net N$20: track 40.1 -> 40.9 mm
- net N$23: track 20.2 -> 19.4 mm
- net N$21: track 53.7 -> 54.4 mm
- net N$16: track 17.2 -> 17.9 mm
Other:
- board text added: "(c) luni 2020-02"
- board text added: "ENC_BOARD_V01"
- board text removed: "ENC_BOARD_V01 (c) luni 2020-02"
